Commit message: draco3 mesh & urdf file updated

File: robot_model/draco/draco.urdf (robot description, URDF)
Before this commit: robot draco, 40 links, 39 joints
Links:
- link neck_pitch_link: geometry visual mesh filename=package://meshes/neck_pitch_link_modified.obj
- link torso_link: geometry visual mesh filename=package://meshes/torso_link.stl

File: robot_model/draco/draco2.urdf (robot description, URDF)
Before this commit: robot draco, 40 links, 39 joints
Links:
- link l_hip_fe_link: geometry visual mesh filename=package://meshes/l_hip_fe_link3.obj
- link l_knee_fe_ld: geometry visual mesh filename=package://meshes/l_knee_fe_ld3.obj
- link l_shoulder_ie_link: geometry visual mesh filename=package://meshes/l_shoulder_ie_link3.obj
- link neck_pitch_link: geometry visual mesh filename=package://meshes/neck_pitch_link3.obj
- link r_hip_fe_link: geometry visual mesh filename=package://meshes/r_hip_fe_link3.obj
- link r_knee_fe_ld: geometry visual mesh filename=package://meshes/r_knee_fe_ld3.obj
- link r_shoulder_ie_link: geometry visual mesh filename=package://meshes/r_shoulder_ie_link3.obj
- link torso_link: geometry visual mesh filename=package://meshes/torso_link3.obj
