Commit message: fixed proto bug and added swing action

File: robot_model/draco/draco_point_contact.urdf (robot description, URDF)
Before this commit: robot draco, 48 links, 47 joints
Links:
- link r_hip_ie_link: geometry collision mesh filename=package://meshes/torso_link3.obj; visual mesh filename=package://meshes/r_hip_ie_link.stl

File: robot_model/draco/draco_point_contact_fb.urdf (robot description, URDF)
Before this commit: robot draco, 49 links, 48 joints
Joints:
- joint base_joint: origin xyz=0 0 0.72 rpy=0 0 0 -> xyz=-0.05 -0.1 0.742691 rpy=0 0 0

Commit message: swing simulation working!

File: robot_model/draco/draco_point_contact.urdf (robot description, URDF)
Before this commit: robot draco, 48 links, 47 joints
Joints:
- joint l_foot_contact_frame_lower_left: origin xyz=-0.1 0.05 0.0 rpy=0 0 0 -> xyz=-0.08 0.04 0.0 rpy=0 0 0
- joint l_foot_contact_frame_lower_right: origin xyz=-0.1 -0.05 0.0 rpy=0 0 0 -> xyz=-0.08 -0.04 0.0 rpy=0 0 0
- joint l_foot_contact_frame_upper_left: origin xyz=0.1 0.05 0.0 rpy=0 0 0 -> xyz=0.08 0.04 0.0 rpy=0 0 0
- joint l_foot_contact_frame_upper_right: origin xyz=0.1 -0.05 0.0 rpy=0 0 0 -> xyz=0.08 -0.04 0.0 rpy=0 0 0
- joint r_foot_contact_frame_lower_left: origin xyz=-0.1 0.05 0.0 rpy=0 0 0 -> xyz=-0.08 0.04 0.0 rpy=0 0 0
- joint r_foot_contact_frame_lower_right: origin xyz=-0.1 -0.05 0.0 rpy=0 0 0 -> xyz=-0.08 -0.04 0.0 rpy=0 0 0
- joint r_foot_contact_frame_upper_left: origin xyz=0.1 0.05 0.0 rpy=0 0 0 -> xyz=0.08 0.04 0.0 rpy=0 0 0
- joint r_foot_contact_frame_upper_right: origin xyz=0.1 -0.05 0.0 rpy=0 0 0 -> xyz=0.08 -0.04 0.0 rpy=0 0 0

File: robot_model/draco/draco_point_contact_fb.urdf (robot description, URDF)
Before this commit: robot draco, 49 links, 48 joints
Joints:
- joint base_joint: origin xyz=-0.05 -0.1 0.742691 rpy=0 0 0 -> xyz=0 0 0.742691 rpy=0 0 0
- joint l_foot_contact_frame_lower_left: origin xyz=-0.1 0.05 0.0 rpy=0 0 0 -> xyz=-0.08 0.04 0.0 rpy=0 0 0
- joint l_foot_contact_frame_lower_right: origin xyz=-0.1 -0.05 0.0 rpy=0 0 0 -> xyz=-0.08 -0.04 0.0 rpy=0 0 0
- joint l_foot_contact_frame_upper_left: origin xyz=0.1 0.05 0.0 rpy=0 0 0 -> xyz=0.08 0.04 0.0 rpy=0 0 0
- joint l_foot_contact_frame_upper_right: origin xyz=0.1 -0.05 0.0 rpy=0 0 0 -> xyz=0.08 -0.04 0.0 rpy=0 0 0
- joint r_foot_contact_frame_lower_left: origin xyz=-0.1 0.05 0.0 rpy=0 0 0 -> xyz=-0.08 0.04 0.0 rpy=0 0 0
- joint r_foot_contact_frame_lower_right: origin xyz=-0.1 -0.05 0.0 rpy=0 0 0 -> xyz=-0.08 -0.04 0.0 rpy=0 0 0
- joint r_foot_contact_frame_upper_left: origin xyz=0.1 0.05 0.0 rpy=0 0 0 -> xyz=0.08 0.04 0.0 rpy=0 0 0
- joint r_foot_contact_frame_upper_right: origin xyz=0.1 -0.05 0.0 rpy=0 0 0 -> xyz=0.08 -0.04 0.0 rpy=0 0 0
