Commit message: draco collocated urdf

File: robot_model/draco/draco_ik_collocated.urdf (robot description, URDF)
Before this commit: robot draco, 40 links, 39 joints
Links:
- link l_hip_fe_link: mass 3.0 -> 2.0
- link l_knee_fe_ld: mass 4.5 -> 5.5
- link r_hip_fe_link: mass 3.0 -> 5.0
- link r_knee_fe_ld: mass 4.5 -> 5.5
Joints:
- joint l_knee_adj: type revolute -> fixed
- joint l_knee_fe_jd: type fixed -> revolute
- joint l_knee_fe_jp: type fixed -> revolute
- joint r_knee_adj: type revolute -> fixed
- joint r_knee_fe_jd: type fixed -> revolute
- joint r_knee_fe_jp: type fixed -> revolute
