Commit message: Modular scenes for data visualizations (class designations)

File: robot_model/draco/draco_modified_foxglove.urdf (robot description, URDF)
Before this commit: robot draco, 40 links, 39 joints
Links:
- link l_ankle_fe_link: geometry visual mesh filename=file:///home/master/rpc/robot_model/draco/meshes/l_ankle_fe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
- link l_ankle_ie_link: geometry collision box size=0.22 0.092012 0.0045015; visual mesh filename=file:///home/master/rpc/robot_model/draco/meshes/l_ankle_ie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
- link l_elbow_fe_link: geometry visual mesh filename=file:///home/master/rpc/robot_model/draco/meshes/l_elbow_fe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
- link l_hip_aa_link: geometry visual mesh filename=file:///home/master/rpc/robot_model/draco/meshes/l_hip_aa_l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
- link l_hip_fe_link: geometry visual mesh filename=file:///home/master/rpc/robot_model/draco/meshes/l_hip_fe_l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
- link l_hip_ie_link: geometry visual mesh filename=file:///home/master/rpc/robot_model/draco/meshes/l_hip_ie_l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
- link l_knee_adj_link: geometry visual mesh filename=file:///home/master/rpc/robot_model/draco/meshes/l_knee_adj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
- link l_knee_fe_ld: geometry visual mesh filename=file:///home/master/rpc/robot_model/draco/meshes/l_knee_fe_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
- link l_knee_fe_lp: geometry visual mesh filename=file:///home/master/rpc/robot_model/draco/meshes/l_knee_fe_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
- link l_sake_gripper_link: geometry visual mesh filename=file:///home/master/rpc/robot_model/draco/meshes/l_sake_gri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
- link l_shoulder_aa_link: geometry visual mesh filename=file:///home/master/rpc/robot_model/draco/meshes/l_shoulder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
- link l_shoulder_fe_link: geometry visual mesh filename=file:///home/master/rpc/robot_model/draco/meshes/l_shoulder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
- link l_shoulder_ie_link: geometry visual mesh filename=file:///home/master/rpc/robot_model/draco/meshes/l_shoulder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
- link l_wrist_ps_link: geometry visual mesh filename=file:///home/master/rpc/robot_model/draco/meshes/l_wrist_ps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
- link neck_pitch_link: geometry visual mesh filename=file:///home/master/rpc/robot_model/draco/meshes/neck_pitch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
- link r_ankle_fe_link: geometry visual mesh filename=file:///home/master/rpc/robot_model/draco/meshes/r_ankle_fe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
- link r_ankle_ie_link: geometry collision box size=0.22 0.092012 0.0045015; visual mesh filename=file:///home/master/rpc/robot_model/draco/meshes/r_ankle_ie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
- link r_elbow_fe_link: geometry visual mesh filename=file:///home/master/rpc/robot_model/draco/meshes/r_elbow_fe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
- link r_hip_aa_link: geometry visual mesh filename=file:///home/master/rpc/robot_model/draco/meshes/r_hip_aa_l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
- link r_hip_fe_link: geometry visual mesh filename=file:///home/master/rpc/robot_model/draco/meshes/r_hip_fe_l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
- link r_hip_ie_link: geometry visual mesh filename=file:///home/master/rpc/robot_model/draco/meshes/r_hip_ie_l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
- link r_knee_adj_link: geometry visual mesh filename=file:///home/master/rpc/robot_model/draco/meshes/r_knee_adj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
- link r_knee_fe_ld: geometry visual mesh filename=file:///home/master/rpc/robot_model/draco/meshes/r_knee_fe_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
- link r_knee_fe_lp: geometry visual mesh filename=file:///home/master/rpc/robot_model/draco/meshes/r_knee_fe_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
- link r_sake_gripper_link: geometry visual mesh filename=file:///home/master/rpc/robot_model/draco/meshes/r_sake_gri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
- link r_shoulder_aa_link: geometry visual mesh filename=file:///home/master/rpc/robot_model/draco/meshes/r_shoulder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
- link r_shoulder_fe_link: geometry visual mesh filename=file:///home/master/rpc/robot_model/draco/meshes/r_shoulder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
- link r_shoulder_ie_link: geometry visual mesh filename=file:///home/master/rpc/robot_model/draco/meshes/r_shoulder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
- link r_wrist_ps_link: geometry visual mesh filename=file:///home/master/rpc/robot_model/draco/meshes/r_wrist_ps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
- link torso_link: geometry visual mesh filename=file:///home/master/rpc/robot_model/draco/meshes/torso_link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
