Commit message: rotate wrist mount by pi/2 to match real robot config

File: robot_model/draco/draco3_modified_collisions.urdf (robot description, URDF)
Before this commit: robot draco, 40 links, 39 joints
Joints:
- joint l_wrist_mount: origin xyz=0 0 0 rpy=0 0 0 -> xyz=0 0 0 rpy=0 0 1.57079
- joint r_wrist_mount: origin xyz=0 0 0 rpy=0 0 0 -> xyz=0 0 0 rpy=0 0 -1.57079

File: robot_model/draco/draco_modified.urdf (robot description, URDF)
Before this commit: robot draco, 40 links, 39 joints
Joints:
- joint l_wrist_mount: origin xyz=0 0 0 rpy=0 0 0 -> xyz=0 0 0 rpy=0 0 1.57079
- joint r_wrist_mount: origin xyz=0 0 0 rpy=0 0 0 -> xyz=0 0 0 rpy=0 0 -1.57079
