Commit message: testing foxglove web apps

File: robot_model/draco/draco_fox_web.urdf (robot description, URDF)
Before this commit: robot draco, 40 links, 39 joints
Links:
- link l_ankle_fe_link: geometry visual mesh filename=package://meshes/l_ankle_fe_link.stl
- link l_ankle_ie_link: geometry collision box size=0.22 0.092012 0.0045015; visual mesh filename=package://meshes/l_ankle_ie_link_small_foot.stl
- link l_elbow_fe_link: geometry visual mesh filename=package://meshes/l_elbow_fe_link.stl
- link l_hip_aa_link: geometry visual mesh filename=package://meshes/l_hip_aa_link.stl
- link l_hip_fe_link: geometry visual mesh filename=package://meshes/l_hip_fe_link3.obj
- link l_hip_ie_link: geometry visual mesh filename=package://meshes/l_hip_ie_link.stl
- link l_knee_adj_link: geometry visual mesh filename=package://meshes/l_knee_adj_link.stl
- link l_knee_fe_ld: geometry visual mesh filename=package://meshes/l_knee_fe_ld3.obj
- link l_knee_fe_lp: geometry visual mesh filename=package://meshes/l_knee_fe_lp.stl
- link l_sake_gripper_link: geometry visual mesh filename=package://meshes/l_sake_gripper_link.stl
- link l_shoulder_aa_link: geometry visual mesh filename=package://meshes/l_shoulder_aa_link.stl
- link l_shoulder_fe_link: geometry visual mesh filename=package://meshes/l_shoulder_fe_link.stl
- link l_shoulder_ie_link: geometry visual mesh filename=package://meshes/l_shoulder_ie_link3.obj
- link l_wrist_ps_link: geometry visual mesh filename=package://meshes/l_wrist_ps_link.stl
- link neck_pitch_link: geometry visual mesh filename=package://meshes/neck_pitch_link3.obj
- link r_ankle_fe_link: geometry visual mesh filename=package://meshes/r_ankle_fe_link.stl
- link r_ankle_ie_link: geometry collision box size=0.22 0.092012 0.0045015; visual mesh filename=package://meshes/r_ankle_ie_link_small_foot.stl
- link r_elbow_fe_link: geometry visual mesh filename=package://meshes/r_elbow_fe_link.stl
- link r_hip_aa_link: geometry visual mesh filename=package://meshes/r_hip_aa_link.stl
- link r_hip_fe_link: geometry visual mesh filename=package://meshes/r_hip_fe_link3.obj
- link r_hip_ie_link: geometry visual mesh filename=package://meshes/r_hip_ie_link.stl
- link r_knee_adj_link: geometry visual mesh filename=package://meshes/r_knee_adj_link.stl
- link r_knee_fe_ld: geometry visual mesh filename=package://meshes/r_knee_fe_ld3.obj
- link r_knee_fe_lp: geometry visual mesh filename=package://meshes/r_knee_fe_lp.stl
- link r_sake_gripper_link: geometry visual mesh filename=package://meshes/r_sake_gripper_link.stl
- link r_shoulder_aa_link: geometry visual mesh filename=package://meshes/r_shoulder_aa_link.stl
- link r_shoulder_fe_link: geometry visual mesh filename=package://meshes/r_shoulder_fe_link.stl
- link r_shoulder_ie_link: geometry visual mesh filename=package://meshes/r_shoulder_ie_link3.obj
- link r_wrist_ps_link: geometry visual mesh filename=package://meshes/r_wrist_ps_link.stl

Commit message: testing foxglove web apps

File: robot_model/draco/draco_fox_web.urdf (robot description, URDF)
Before this commit: robot draco, 40 links, 39 joints
Links:
- link torso_link: geometry visual mesh filename=https://raw.githubusercontent.com/shbang91/rpc/feature/foxg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

Commit message: visualization in foxglove web

File: robot_model/draco/draco_fox_web.urdf (robot description, URDF)
Before this commit: robot draco, 40 links, 39 joints
Links:
- link l_ankle_fe_link: geometry visual mesh filename=https://raw.githubusercontent.com/shbang91/rpc/feature/foxg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
- link l_ankle_ie_link: geometry collision box size=0.22 0.092012 0.0045015; visual mesh filename=https://raw.githubusercontent.com/shbang91/rpc/feature/foxg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
- link l_elbow_fe_link: geometry visual mesh filename=https://raw.githubusercontent.com/shbang91/rpc/feature/foxg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
- link l_hip_aa_link: geometry visual mesh filename=https://raw.githubusercontent.com/shbang91/rpc/feature/foxg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
- link l_hip_fe_link: geometry visual mesh filename=https://raw.githubusercontent.com/shbang91/rpc/feature/foxg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
- link l_hip_ie_link: geometry visual mesh filename=https://raw.githubusercontent.com/shbang91/rpc/feature/foxg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
- link l_knee_adj_link: geometry visual mesh filename=https://raw.githubusercontent.com/shbang91/rpc/feature/foxg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
- link l_knee_fe_ld: geometry visual mesh filename=https://raw.githubusercontent.com/shbang91/rpc/feature/foxg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
- link l_knee_fe_lp: geometry visual mesh filename=https://raw.githubusercontent.com/shbang91/rpc/feature/foxg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
- link l_sake_gripper_link: geometry visual mesh filename=https://raw.githubusercontent.com/shbang91/rpc/feature/foxg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
- link l_shoulder_aa_link: geometry visual mesh filename=https://raw.githubusercontent.com/shbang91/rpc/feature/foxg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
- link l_shoulder_fe_link: geometry visual mesh filename=https://raw.githubusercontent.com/shbang91/rpc/feature/foxg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
- link l_shoulder_ie_link: geometry visual mesh filename=https://raw.githubusercontent.com/shbang91/rpc/feature/foxg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
- link l_wrist_ps_link: geometry visual mesh filename=https://raw.githubusercontent.com/shbang91/rpc/feature/foxg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
- link neck_pitch_link: geometry visual mesh filename=https://raw.githubusercontent.com/shbang91/rpc/feature/foxg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
- link r_ankle_fe_link: geometry visual mesh filename=https://raw.githubusercontent.com/shbang91/rpc/feature/foxg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
- link r_ankle_ie_link: geometry collision box size=0.22 0.092012 0.0045015; visual mesh filename=https://raw.githubusercontent.com/shbang91/rpc/feature/foxg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
- link r_elbow_fe_link: geometry visual mesh filename=https://raw.githubusercontent.com/shbang91/rpc/feature/foxg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
- link r_hip_aa_link: geometry visual mesh filename=https://raw.githubusercontent.com/shbang91/rpc/feature/foxg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
- link r_hip_fe_link: geometry visual mesh filename=https://raw.githubusercontent.com/shbang91/rpc/feature/foxg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
- link r_hip_ie_link: geometry visual mesh filename=https://raw.githubusercontent.com/shbang91/rpc/feature/foxg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
- link r_knee_adj_link: geometry visual mesh filename=https://raw.githubusercontent.com/shbang91/rpc/feature/foxg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
- link r_knee_fe_ld: geometry visual mesh filename=https://raw.githubusercontent.com/shbang91/rpc/feature/foxg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
- link r_knee_fe_lp: geometry visual mesh filename=https://raw.githubusercontent.com/shbang91/rpc/feature/foxg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
- link r_sake_gripper_link: geometry visual mesh filename=https://raw.githubusercontent.com/shbang91/rpc/feature/foxg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
- link r_shoulder_aa_link: geometry visual mesh filename=https://raw.githubusercontent.com/shbang91/rpc/feature/foxg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
- link r_shoulder_fe_link: geometry visual mesh filename=https://raw.githubusercontent.com/shbang91/rpc/feature/foxg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
- link r_shoulder_ie_link: geometry visual mesh filename=https://raw.githubusercontent.com/shbang91/rpc/feature/foxg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
- link r_wrist_ps_link: geometry visual mesh filename=https://raw.githubusercontent.com/shbang91/rpc/feature/foxg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
