Commit message: visualization in foxglove web

File: robot_model/draco/draco_fox_web_old.urdf (robot description, URDF)
Before this commit: robot draco, 40 links, 39 joints
Links:
- link l_ankle_fe_link: geometry visual mesh filename=https://raw.githubusercontent.com/shbang91/rpc/feature/foxg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
- link l_ankle_ie_link: geometry collision box size=0.22 0.092012 0.0045015; visual mesh filename=https://raw.githubusercontent.com/shbang91/rpc/feature/foxg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
- link l_elbow_fe_link: geometry visual mesh filename=https://raw.githubusercontent.com/shbang91/rpc/feature/foxg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
- link l_hip_aa_link: geometry visual mesh filename=https://raw.githubusercontent.com/shbang91/rpc/feature/foxg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
- link l_hip_fe_link: geometry visual mesh filename=https://raw.githubusercontent.com/shbang91/rpc/feature/foxg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
- link l_hip_ie_link: geometry visual mesh filename=https://raw.githubusercontent.com/shbang91/rpc/feature/foxg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
- link l_knee_adj_link: geometry visual mesh filename=https://raw.githubusercontent.com/shbang91/rpc/feature/foxg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
- link l_knee_fe_ld: geometry visual mesh filename=https://raw.githubusercontent.com/shbang91/rpc/feature/foxg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
- link l_knee_fe_lp: geometry visual mesh filename=https://raw.githubusercontent.com/shbang91/rpc/feature/foxg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
- link l_sake_gripper_link: geometry visual mesh filename=https://raw.githubusercontent.com/shbang91/rpc/feature/foxg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
- link l_shoulder_aa_link: geometry visual mesh filename=https://raw.githubusercontent.com/shbang91/rpc/feature/foxg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
- link l_shoulder_fe_link: geometry visual mesh filename=https://raw.githubusercontent.com/shbang91/rpc/feature/foxg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
- link l_shoulder_ie_link: geometry visual mesh filename=https://raw.githubusercontent.com/shbang91/rpc/feature/foxg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
- link l_wrist_ps_link: geometry visual mesh filename=https://raw.githubusercontent.com/shbang91/rpc/feature/foxg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
- link neck_pitch_link: geometry visual mesh filename=https://raw.githubusercontent.com/shbang91/rpc/feature/foxg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
- link r_ankle_fe_link: geometry visual mesh filename=https://raw.githubusercontent.com/shbang91/rpc/feature/foxg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
- link r_ankle_ie_link: geometry collision box size=0.22 0.092012 0.0045015; visual mesh filename=https://raw.githubusercontent.com/shbang91/rpc/feature/foxg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
- link r_elbow_fe_link: geometry visual mesh filename=https://raw.githubusercontent.com/shbang91/rpc/feature/foxg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
- link r_hip_aa_link: geometry visual mesh filename=https://raw.githubusercontent.com/shbang91/rpc/feature/foxg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
- link r_hip_fe_link: geometry visual mesh filename=https://raw.githubusercontent.com/shbang91/rpc/feature/foxg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
- link r_hip_ie_link: geometry visual mesh filename=https://raw.githubusercontent.com/shbang91/rpc/feature/foxg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
- link r_knee_adj_link: geometry visual mesh filename=https://raw.githubusercontent.com/shbang91/rpc/feature/foxg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
- link r_knee_fe_ld: geometry visual mesh filename=https://raw.githubusercontent.com/shbang91/rpc/feature/foxg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
- link r_knee_fe_lp: geometry visual mesh filename=https://raw.githubusercontent.com/shbang91/rpc/feature/foxg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
- link r_sake_gripper_link: geometry visual mesh filename=https://raw.githubusercontent.com/shbang91/rpc/feature/foxg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
- link r_shoulder_aa_link: geometry visual mesh filename=https://raw.githubusercontent.com/shbang91/rpc/feature/foxg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
- link r_shoulder_fe_link: geometry visual mesh filename=https://raw.githubusercontent.com/shbang91/rpc/feature/foxg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
- link r_shoulder_ie_link: geometry visual mesh filename=https://raw.githubusercontent.com/shbang91/rpc/feature/foxg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
- link r_wrist_ps_link: geometry visual mesh filename=https://raw.githubusercontent.com/shbang91/rpc/feature/foxg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
- link torso_link: geometry visual mesh filename=https://raw.githubusercontent.com/shbang91/rpc/feature/foxg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
