Commit message: updated draco new feets mass

File: robot_model/draco/draco_modified.urdf (robot description, URDF)
Before this commit: robot draco, 40 links, 39 joints
Links:
- link l_ankle_ie_link: mass 0.478 -> 0.901
- link r_ankle_ie_link: mass 0.478 -> 0.901

Commit message: draco small feet urdf updated

File: robot_model/draco/draco_modified.urdf (robot description, URDF)
Before this commit: robot draco, 40 links, 39 joints
Links:
- link l_ankle_ie_link: mass 0.901 -> 0.478
- link r_ankle_ie_link: mass 0.901 -> 0.478

Commit message: added F/T sensor
ankle_ie inertia needs to be updated

File: robot_model/draco/draco_modified.urdf (robot description, URDF)
Before this commit: robot draco, 40 links, 39 joints
Links:
- link l_ankle_ie_link: mass 0.478 -> 0.5917
- link r_ankle_ie_link: mass 0.478 -> 0.5917

Commit message: updated urdf model with f/t sensor
intertia parameter needs to be updated

File: robot_model/draco/draco_modified.urdf (robot description, URDF)
Before this commit: robot draco, 40 links, 39 joints
Links:
- link l_ankle_ie_link: geometry collision box size=0.2 0.1 0.0664; visual mesh filename=package://meshes/l_ankle_ie_link.stl
- link r_ankle_ie_link: geometry collision box size=0.2 0.1 0.0664; visual mesh filename=package://meshes/r_ankle_ie_link.stl
Joints:
- joint l_foot_contact_frame: origin xyz=0 0 -0.076 rpy=0 0 0 -> xyz=0 0 -0.0833 rpy=0 0 0
- joint r_foot_contact_frame: origin xyz=0 0 -0.076 rpy=0 0 0 -> xyz=0 0 -0.0833 rpy=0 0 0

Commit message: changed foot collision origin for sim

File: robot_model/draco/draco_modified.urdf (robot description, URDF)
Before this commit: robot draco, 40 links, 39 joints
Links:
- link l_ankle_ie_link: geometry collision box size=0.2 0.1 0.0591; visual mesh filename=package://meshes/l_ankle_ie_link.stl
- link r_ankle_ie_link: geometry collision box size=0.2 0.1 0.0591; visual mesh filename=package://meshes/r_ankle_ie_link.stl

Commit message: stabilized the robot with some gain tuning after F/T sensors implementation

File: robot_model/draco/draco_modified.urdf (robot description, URDF)
Before this commit: robot draco, 40 links, 39 joints
Links:
- link l_ankle_ie_link: mass 0.478 -> 0.5917
- link r_ankle_ie_link: mass 0.478 -> 0.5917
Joints:
- joint l_foot_contact_frame: origin xyz=0 0 -0.076 rpy=0 0 0 -> xyz=0 0 -0.0833 rpy=0 0 0
- joint r_foot_contact_frame: origin xyz=0 0 -0.076 rpy=0 0 0 -> xyz=0 0 -0.0833 rpy=0 0 0

Commit message: updated URDF model reflecting F/T sensor inclusion

File: robot_model/draco/draco_modified.urdf (robot description, URDF)
Before this commit: robot draco, 40 links, 39 joints
Joints:
- joint l_foot_contact_frame: origin xyz=0 0 -0.076 rpy=0 0 0 -> xyz=0 0 -0.0833 rpy=0 0 0
- joint r_foot_contact_frame: origin xyz=0 0 -0.076 rpy=0 0 0 -> xyz=0 0 -0.0833 rpy=0 0 0

Commit message: added camera link and updated robot model link numbering

File: robot_model/draco/draco_modified.urdf (robot description, URDF)
Before this commit: robot draco, 40 links, 39 joints
Links:
- added link l_multisense_camera, mass 1e-9; visual sphere radius=0.01
Joints:
- added joint neck_to_multisense_camera: type fixed, parent neck_pitch_link, child l_multisense_camera, origin xyz=0 0 0 rpy=0 0 0, axis 0 0 0

Commit message: start using the different URDF that Apptronik gave

File: robot_model/draco/draco_modified.urdf (robot description, URDF)
Before this commit: robot draco, 40 links, 39 joints
Joints:
- joint l_ankle_fe: origin xyz=0 0.00599 -0.248231 rpy=0 0 0 -> xyz=-6.26776e-17 -1.80411e-16 -0.248231 rpy=2.01226e-15 1.44763e-15 -7.77124e-18
- joint l_knee_fe_jd: origin xyz=0.0 0.0 -0.1117386 rpy=0 0 0 -> xyz=0 0.00600074 -0.1117383 rpy=-1.90275e-16 1.31839e-16 2.80923e-17
- joint r_ankle_fe: origin xyz=0 -0.006 -0.248231 rpy=0 0 0 -> xyz=-1.70255e-16 -9.71445e-17 -0.248231 rpy=-1.09947e-29 -6.39256e-14 1.4244e-16
- joint r_knee_fe_jd: origin xyz=0 0 -0.1117386 rpy=0 0 0 -> xyz=0 -0.00600074 -0.1117383 rpy=1.06003e-30 6.64446e-33 -5.70613e-32

Commit message: yamls used for squatting
control com xy & base height

File: robot_model/draco/draco_modified.urdf (robot description, URDF)
Before this commit: robot draco, 40 links, 39 joints
Joints:
- joint l_wrist_mount: origin xyz=0 0 0 rpy=0 0 0 -> xyz=0 0 0 rpy=0 0 1.57
- joint r_wrist_mount: origin xyz=0 0 0 rpy=0 0 0 -> xyz=0 0 0 rpy=0 0 -1.57

Commit message: updated URDF with kinematic and dynamic properties of curved ankle
Updated, on both l_ and r_ankle_ie:
  * joint limits to be within +/- 30 deg, 0 being foot flat horizontally
  * STL files have origin at rotating axis, instead of base of robot
  * collision box covers only the foot, instead of additional height
  * moments of inertia updated w.r.t. CoM
  * contact frames updates with new height and lateral offset

File: robot_model/draco/draco_modified.urdf (robot description, URDF)
Before this commit: robot draco, 40 links, 39 joints
Links:
- link l_ankle_ie_link: geometry collision box size=0.22 0.092012 0.0045015; visual mesh filename=package://meshes/l_ankle_ie_link_small_foot.stl
- link r_ankle_ie_link: geometry collision box size=0.22 0.092012 0.0045015; visual mesh filename=package://meshes/r_ankle_ie_link_small_foot.stl
Joints:
- joint l_ankle_ie: limit lower=-0.785398 upper=0.261799 effort=30 velocity=11.1 -> lower=-0.523599 upper=0.523599 effort=30 velocity=11.1
- joint l_foot_contact_frame: origin xyz=0 0 -0.0833 rpy=0 0 0 -> xyz=0 -0.008432 -0.087801 rpy=0 0 0
- joint r_ankle_ie: limit lower=-0.261799 upper=0.785398 effort=30 velocity=11.1 -> lower=-0.523599 upper=0.523599 effort=30 velocity=11.1
- joint r_foot_contact_frame: origin xyz=0 0 -0.0833 rpy=0 0 0 -> xyz=0 0.008432 -0.087801 rpy=0 0 0

Commit message: initial commit

File: robot_model/draco/draco_modified.urdf (robot description, URDF)
Before this commit: robot draco, 40 links, 39 joints
Links:
- link l_knee_fe_ld: geometry collision sphere radius=0.055; collision sphere radius=0.065
- link r_knee_fe_ld: geometry collision sphere radius=0.055; collision sphere radius=0.065
Joints:
- joint l_wrist_mount: origin xyz=0 0 0 rpy=0 0 1.57079 -> xyz=0 0 0 rpy=0 0 0
- joint r_wrist_mount: origin xyz=0 0 0 rpy=0 0 -1.57079 -> xyz=0 0 0 rpy=0 0 0
