Commit message: updated draco3 model

File: robot_model/draco/draco_latest_collisions.urdf (robot description, URDF)
Before this commit: robot draco, 40 links, 39 joints
Links:
- link l_ankle_fe_link: geometry collision sphere radius=0.055; visual mesh filename=package://meshes/l_ankle_fe_link.stl
- link l_ankle_ie_link: geometry collision box size=0.22 0.1 0.02; visual mesh filename=package://meshes/l_ankle_ie_link_small_foot.stl
- link l_elbow_fe_link: geometry collision sphere radius=0.076; visual mesh filename=package://meshes/l_elbow_fe_link.stl
- link l_hip_aa_link: geometry visual mesh filename=package://meshes/l_hip_aa_link.stl
- link l_hip_fe_link: geometry collision cylinder length=0.243 radius=0.049; collision sphere radius=0.055
- link l_hip_ie_link: geometry visual mesh filename=package://meshes/l_hip_ie_link.stl
- link l_knee_adj_link: geometry visual mesh filename=package://meshes/l_knee_adj_link.stl
- link l_knee_fe_ld: geometry collision cylinder length=0.16 radius=0.055; collision sphere radius=0.055
- link l_knee_fe_lp: geometry visual mesh filename=package://meshes/l_knee_fe_lp.stl
- link l_sake_gripper_link: geometry collision box size=0.06 0.11 0.223; visual mesh filename=package://meshes/l_sake_gripper_link.stl
- link l_shoulder_aa_link: geometry visual mesh filename=package://meshes/l_shoulder_aa_link.stl
- link l_shoulder_fe_link: geometry visual mesh filename=package://meshes/l_shoulder_fe_link.stl
- link l_shoulder_ie_link: geometry collision cylinder length=0.2 radius=0.03; collision sphere radius=0.064
- link l_wrist_ps_link: geometry visual mesh filename=package://meshes/l_wrist_ps_link.stl
- link neck_pitch_link: geometry visual mesh filename=package://meshes/neck_pitch_link3.obj
- link r_ankle_fe_link: geometry collision sphere radius=0.055; visual mesh filename=package://meshes/r_ankle_fe_link.stl
- link r_ankle_ie_link: geometry collision box size=0.22 0.1 0.02; visual mesh filename=package://meshes/r_ankle_ie_link_small_foot.stl
- link r_elbow_fe_link: geometry collision sphere radius=0.076; visual mesh filename=package://meshes/r_elbow_fe_link.stl
- link r_hip_aa_link: geometry visual mesh filename=package://meshes/r_hip_aa_link.stl
- link r_hip_fe_link: geometry collision cylinder length=0.243 radius=0.049; collision sphere radius=0.055
- link r_hip_ie_link: geometry visual mesh filename=package://meshes/r_hip_ie_link.stl
- link r_knee_adj_link: geometry visual mesh filename=package://meshes/r_knee_adj_link.stl
- link r_knee_fe_ld: geometry collision cylinder length=0.16 radius=0.055; collision sphere radius=0.055
- link r_knee_fe_lp: geometry visual mesh filename=package://meshes/r_knee_fe_lp.stl
- link r_sake_gripper_link: geometry collision box size=0.06 0.11 0.223; visual mesh filename=package://meshes/r_sake_gripper_link.stl
- link r_shoulder_aa_link: geometry visual mesh filename=package://meshes/r_shoulder_aa_link.stl
- link r_shoulder_fe_link: geometry visual mesh filename=package://meshes/r_shoulder_fe_link.stl
- link r_shoulder_ie_link: geometry collision cylinder length=0.2 radius=0.03; collision sphere radius=0.064
- link r_wrist_ps_link: geometry visual mesh filename=package://meshes/r_wrist_ps_link.stl
- link torso_link: geometry collision box size=0.122 0.191 0.3575; visual mesh filename=package://meshes/torso_link3.obj
Joints:
- joint l_foot_contact_frame: origin xyz=0 -0.008432 -0.087801 rpy=0 0 0 -> xyz=0 0 -0.0932995 rpy=0 0 0
- joint r_foot_contact_frame: origin xyz=0 0.008432 -0.087801 rpy=0 0 0 -> xyz=0 0 -0.0932995 rpy=0 0 0

Commit message: update draco mujoco model

File: robot_model/draco/draco_latest_collisions.urdf (robot description, URDF)
Before this commit: robot draco, 40 links, 39 joints
Links:
- link l_ankle_ie_link: geometry collision box size=0.22 0.1 0.009; visual mesh filename=package://meshes/l_ankle_ie_link_small_foot.stl
- link r_ankle_ie_link: geometry collision box size=0.22 0.1 0.009; visual mesh filename=package://meshes/r_ankle_ie_link_small_foot.stl
Joints:
- joint l_foot_contact_frame: origin xyz=0 0 -0.0932995 rpy=0 0 0 -> xyz=0 0 -0.0877995 rpy=0 0 0
- joint r_foot_contact_frame: origin xyz=0 0 -0.0932995 rpy=0 0 0 -> xyz=0 0 -0.0877995 rpy=0 0 0
