Commit message: ICRA CII analysis added

File: robot_model/hubo/URDF_HuboPlus_Float_2.urdf (robot description, URDF)
Before this commit: robot huboplus, 61 links, 60 joints
Links:
- link Body_HNP: geometry visual box size=0.2 0.1 0.0591
- link Body_Hip: geometry visual box size=0.2 0.1 0.0591
- link Body_LAP: geometry visual box size=0.2 0.1 0.0591
- link Body_LAR: geometry visual box size=0.2 0.1 0.0591
- link Body_LEP: geometry visual box size=0.2 0.1 0.0591
- link Body_LHP: geometry visual box size=0.2 0.1 0.0591
- link Body_LHR: geometry visual box size=0.2 0.1 0.0591
- link Body_LHY: geometry visual box size=0.2 0.1 0.0591
- link Body_LKP: geometry visual box size=0.2 0.1 0.0591
- link Body_LSP: geometry visual box size=0.2 0.1 0.0591
- link Body_LSR: geometry visual box size=0.2 0.1 0.0591
- link Body_LSY: geometry visual box size=0.2 0.1 0.0591
- link Body_LWP: geometry visual box size=0.2 0.1 0.0591
- link Body_LWY: geometry visual box size=0.2 0.1 0.0591
- link Body_RAP: geometry visual box size=0.2 0.1 0.0591
- link Body_RAR: geometry visual box size=0.2 0.1 0.0591
- link Body_REP: geometry visual box size=0.2 0.1 0.0591
- link Body_RHP: geometry visual box size=0.2 0.1 0.0591
- link Body_RHR: geometry visual box size=0.2 0.1 0.0591
- link Body_RKP: geometry visual box size=0.2 0.1 0.0591
- link Body_RSP: geometry visual box size=0.2 0.1 0.0591
- link Body_RSR: geometry visual box size=0.2 0.1 0.0591
- link Body_RSY: geometry visual box size=0.2 0.1 0.0591
- link Body_RWP: geometry visual box size=0.2 0.1 0.0591
- link Body_RWY: geometry visual box size=0.2 0.1 0.0591
- link Body_Torso: geometry visual box size=0.2 0.1 0.0591
- link leftIndexDistal: geometry visual box size=0.2 0.1 0.0591
- link leftIndexMedial: geometry visual box size=0.2 0.1 0.0591
- link leftIndexProximal: geometry visual box size=0.2 0.1 0.0591
- link leftMiddleDistal: geometry visual box size=0.2 0.1 0.0591
- link leftMiddleMedial: geometry visual box size=0.2 0.1 0.0591
- link leftPinkyDistal: geometry visual box size=0.2 0.1 0.0591
- link leftPinkyMedial: geometry visual box size=0.2 0.1 0.0591
- link leftPinkyProximal: geometry visual box size=0.2 0.1 0.0591
- link leftRingDistal: geometry visual box size=0.2 0.1 0.0591
- link leftRingMedial: geometry visual box size=0.2 0.1 0.0591
- link leftRingProximal: geometry visual box size=0.2 0.1 0.0591
- link leftThumbDistal: geometry visual box size=0.2 0.1 0.0591
- link leftThumbProximal: geometry visual box size=0.2 0.1 0.0591
- link rightIndexMedial: geometry visual box size=0.2 0.1 0.0591
- link rightMiddleDistal: geometry visual box size=0.2 0.1 0.0591
- link rightMiddleMedial: geometry visual box size=0.2 0.1 0.0591
- link rightMiddleProximal: geometry visual box size=0.2 0.1 0.0591
- link rightPinkyDistal: geometry visual box size=0.2 0.1 0.0591
- link rightPinkyMedial: geometry visual box size=0.2 0.1 0.0591
- link rightPinkyProximal: geometry visual box size=0.2 0.1 0.0591
- link rightRingDistal: geometry visual box size=0.2 0.1 0.0591
- link rightRingMedial: geometry visual box size=0.2 0.1 0.0591
- link rightThumbDistal: geometry visual box size=0.2 0.1 0.0591
