Commit message: atlas crbi trainer fix

File: robot_model/atlas/atlas.urdf (robot description, URDF)
Before this commit: robot multisense_sl, 34 links, 33 joints
Links:
- link l_larm: geometry collision box size=0.135 0.15 0.06; collision cylinder length=0.125 radius=0.045
- link l_lfarm: geometry collision box size=0.13 0.09 0.07; collision cylinder length=0.05 radius=0.03
- link l_ufarm: geometry collision box size=0.135 0.1 0.045; collision cylinder length=0.125 radius=0.045
- link r_larm: geometry collision box size=0.135 0.15 0.06; collision cylinder length=0.125 radius=0.045
- link r_lfarm: geometry collision box size=0.13 0.09 0.07; collision cylinder length=0.05 radius=0.03
- link r_ufarm: geometry collision box size=0.135 0.1 0.045; collision cylinder length=0.125 radius=0.045
