Commit message: optimo summon without cmd

File: robot_model/optimo/optimo.xacro (robot description, xacro)
@@ -293,83 +293,3 @@
         </collision>
     </link>
-    <!-- Gazebo stuff-->
-    <ros2_control name="IgnitionSystem" type="system">
-        <hardware>
-            <plugin>ign_ros2_control/IgnitionSystem</plugin>
-        </hardware>
-        <joint name="joint1">
-            <command_interface name="effort">
-                <param name="min">-150</param>
-                <param name="max">150</param>
-            </command_interface>
-            <state_interface name="position"/>
-            <state_interface name="velocity" />
-            <state_interface name="effort" />
-        </joint>
-        <joint name="joint2">
-            <command_interface name="effort">
-                <param name="min">-150</param>
-                <param name="max">150</param>
-            </command_interface>
-            <state_interface name="position">
-            </state_interface>
-            <state_interface name="velocity" />
-            <state_interface name="effort" />
-        </joint>
-        <joint name="joint3">
-            <command_interface name="effort">
-                <param name="min">-150</param>
-                <param name="max">150</param>
-            </command_interface>
-            <state_interface name="position"/>
-            <state_interface name="velocity" />
-            <state_interface name="effort" />
-        </joint>
-        <joint name="joint4">
-            <command_interface name="effort">
-                <param name="min">-150</param>
-                <param name="max">150</param>
-            </command_interface>
-            <state_interface name="position"/>
-            <state_interface name="velocity" />
-            <state_interface name="effort" />
-        </joint>
-        <joint name="joint5">
-            <command_interface name="effort">
-                <param name="min">-150</param>
-                <param name="max">150</param>
-            </command_interface>
-            <state_interface name="position"/>
-            <state_interface name="velocity" />
-            <state_interface name="effort" />
-        </joint>
-        <joint name="joint6">
-            <command_interface name="effort">
-                <param name="min">-150</param>
-                <param name="max">150</param>
-            </command_interface>
-            <state_interface name="position"/>
-            <state_interface name="velocity" />
-            <state_interface name="effort" />
-        </joint>
-        <joint name="joint7">
-            <command_interface name="effort">
-                <param name="min">-150</param>
-                <param name="max">150</param>
-            </command_interface>
-            <state_interface name="position"/>
-            <state_interface name="velocity" />
-            <state_interface name="effort" />
-        </joint>
-    </ros2_control>
-    <gazebo>
-        <!-- Joint state publisher -->
-        <plugin filename="ign_ros2_control-system" name="ign_ros2_control::IgnitionROS2ControlPlugin">
-            <!-- need to make $(find optimo_sim) work again...-->
-            <parameters>$(find optimo_sim)/config/control.yaml</parameters>
-        </plugin>
-        <plugin filename="MechanicalStop" name="optimo_ros::MechanicalStop">
-            <init_pos>0 3.3 0 -2.36 0 -1.13 1.57</init_pos>
-        </plugin>
-    </gazebo>
 </robot>
