Commit message: urdf gazebo param deleted

File: robot_model/optimo/optimo.urdf (robot description, URDF)
Before this commit: robot optimo, 18 links, 17 joints
Links:
- removed link world
- link ee: geometry 
- link link1: mass None -> 0.00
- link link2: mass None -> 0.00
- link link3: mass None -> 0.00
- link link4: mass None -> 0.00
- link link5: mass None -> 0.00
- link link6: mass None -> 0.00
- link link7: mass None -> 0.00
- link stand: mass None -> 1
Joints:
- removed joint world_to_stand
- joint stand_to_link0: origin xyz=0 0 .27 rpy=0 0 0 -> xyz=0 0 .77 rpy=0 0 0

File: robot_model/optimo/optimo.xacro (robot description, xacro)
@@ -8,14 +8,8 @@
         <color rgba="0.5 0.5 1 1.0"/>
     </material>
-    <!-- Used for fixing robot to Gazebo 'base_link' -->
-    <link name="world" />
-    <joint name="world_to_stand" type="fixed">
-        <parent link="world"/>
-        <child link="stand"/>
-        <origin xyz="0 0 1" rpy="0 0 0"/>
-    </joint>
+    <!-- Robot Pedestal -->
     <link name="stand">
         <visual>
-            <origin xyz="0 0 -0.5" rpy="0 0 0"/>
+            <origin xyz="0 0 0.0" rpy="0 0 0"/>
             <geometry>
                 <box size="0.3 0.3 1"/>
@@ -24,9 +18,14 @@
         </visual>
         <collision>
-            <origin xyz="0 0 -0.5" rpy="0 0 0"/>
+            <origin xyz="0 0 0.0" rpy="0 0 0"/>
             <geometry>
                 <box size="0.3 0.3 1"/>
             </geometry>
         </collision>
+        <inertial>
+            <origin xyz="0 0 0.0" rpy="0 0 0"/>
+            <mass value="1"/>
+            <inertia ixx="0.1" ixy="0.0" ixz="0.0" iyy="0.1" iyz="0.0" izz="0.1"/>
+        </inertial>
     </link>
     <joint name="stand_to_link0" type="fixed">
@@ -34,5 +33,5 @@
         <child link="link0" />
         <!-- .27 puts the link on the stand -->
-        <origin xyz="0 0 .27" rpy="0 0 0" />
+        <origin xyz="0 0 .77" rpy="0 0 0" />
     </joint>
     <!-- Base Link -->
@@ -52,8 +51,15 @@
             <origin xyz="0 0 0" />
             <mass value="1" />
-            <inertia ixx="0" ixy="0.0" ixz="0.0" iyy="0" iyz="0.0" izz="0" />
-        </inertial>
-    </link>
-    <link name="link1" />
+            <inertia ixx="0.1" ixy="0.1" ixz="0.0" iyy="0.1" iyz="0.0" izz="0" />
+        </inertial>
+    </link>
+    <!-- Link 1 -->
+    <link name="link1">
+         <inertial>
+            <origin xyz="0 0 0" />
+            <mass value="0.00" />
+            <inertia ixx="0.0" ixy="0.0" ixz="0.0" iyy="0.0" iyz="0.0" izz="0.0" />
+        </inertial>
+    </link>
     <joint name="joint1" type="revolute">
         <origin xyz="0 0 0" rpy="0 0 0" />
@@ -87,5 +93,12 @@
         </inertial>
     </link>
-    <link name="link2" />
+    <!-- Link 2 -->
+    <link name="link2">
+        <inertial>
+            <origin xyz="0 0 0" />
+            <mass value="0.00" />
+            <inertia ixx="0.0" ixy="0.0" ixz="0.0" iyy="0.0" iyz="0.0" izz="0.0" />
+        </inertial>
+    </link>
     <joint name="joint2" type="revolute">
         <origin xyz="0 0 0" rpy="0 0 0" />
@@ -119,5 +132,12 @@
         </inertial>
     </link>
-    <link name="link3" />
+    <!-- Link 3 -->
+    <link name="link3" >
+        <inertial>
+            <origin xyz="0 0 0" />
+            <mass value="0.00" />
+            <inertia ixx="0.0" ixy="0.0" ixz="0.0" iyy="0.0" iyz="0.0" izz="0.0" />
+        </inertial>
+    </link>
     <joint name="joint3" type="revolute">
         <origin xyz="0 0 0.4" rpy="0 0 0" />
@@ -152,5 +172,12 @@
         </inertial>
     </link>
-    <link name="link4" />
+    <!-- Link 4 -->
+    <link name="link4" >
+        <inertial>
+            <origin xyz="0 0 0" />
+            <mass value="0.00" />
+            <inertia ixx="0.0" ixy="0.0" ixz="0.0" iyy="0.0" iyz="0.0" izz="0.0" />
+        </inertial>
+    </link>
     <joint name="joint4" type="revolute">
         <origin xyz="0 0 0" rpy="0 0 0" />
@@ -184,5 +211,12 @@
         </inertial>
     </link>
-    <link name="link5" />
+    <!-- Link 5 -->
+    <link name="link5" >
+        <inertial>
+            <origin xyz="0 0 0" />
+            <mass value="0.00" />
+            <inertia ixx="0.0" ixy="0.0" ixz="0.0" iyy="0.0" iyz="0.0" izz="0.0" />
+        </inertial>
+    </link>
     <joint name="joint5" type="revolute">
         <origin xyz="0 0 0.4" rpy="0 0 0" />
@@ -216,5 +250,12 @@
         </inertial>
     </link>
-    <link name="link6" />
+    <!-- Link 6 -->
+    <link name="link6" >
+        <inertial>
+            <origin xyz="0 0 0" />
+            <mass value="0.00" />
+            <inertia ixx="0.0" ixy="0.0" ixz="0.0" iyy="0.0" iyz="0.0" izz="0.0" />
+        </inertial>
+    </link>
     <joint name="joint6" type="revolute">
         <origin xyz="0 0 0" rpy="0 0 0" />
@@ -248,5 +289,12 @@
         </inertial>
     </link>
-    <link name="link7" />
+    <!-- Link 7 -->
+    <link name="link7" >
+        <inertial>
+            <origin xyz="0 0 0" />
+            <mass value="0.00" />
+            <inertia ixx="0.0" ixy="0.0" ixz="0.0" iyy="0.0" iyz="0.0" izz="0.0" />
+        </inertial>
+    </link>
     <joint name="joint7" type="revolute">
         <origin xyz="0 0 0" rpy="0 0 0" />
@@ -280,4 +328,5 @@
         </inertial>
     </link>
+    <!-- End Effector -->
     <joint name="ee_joint" type="fixed">
         <origin xyz="0 0 0.33" rpy="0 0 0" />
@@ -286,10 +335,9 @@
     </joint>
     <link name="ee">
-        <collision>
-            <origin xyz="0 0 -0.075" rpy="0 0 0"/>
-            <geometry>
-                <box size="0.1 0.1 0.15"/>
-            </geometry>
-        </collision>
+        <inertia>
+            <origin xyz="0 0 0" rpy="0 0 0"/>
+            <mass value="0.00"/>
+            <inertia ixx="0.0" ixy="0.0" ixz="0.0" iyy="0.0" iyz="0.0" izz="0.0"/>
+        </inertia>
     </link>
 </robot>

Commit message: wip

File: robot_model/optimo/optimo.urdf (robot description, URDF)
Before this commit: robot optimo, 17 links, 16 joints
Links:
- removed link ee
- removed link link0
- removed link link1
- removed link link1_passive
- removed link link2
- removed link link2_passive
- removed link link3
- removed link link3_passive
- removed link link4
- removed link link4_passive
- removed link link5
- removed link link5_passive
- removed link link6
- removed link link6_passive
- removed link link7
- removed link link7_passive
- removed link stand
- added link optimo_base_link, mass 0.0; visual sphere radius=0.01
- added link optimo_ee_link, mass 0.0
- added link optimo_link0, mass 1; collision mesh filename=package://meshes/col0.stl; visual mesh filename=package://meshes/link0.stl
- added link optimo_link1, mass 0.0
- added link optimo_link1_passive, mass 4.152; collision mesh filename=package://meshes/col1.stl; visual mesh filename=package://meshes/link1.stl
- added link optimo_link2, mass 0.0
- added link optimo_link2_passive, mass 1.72; collision mesh filename=package://meshes/col2.stl; visual mesh filename=package://meshes/link2.stl
- added link optimo_link3, mass 0.0
- added link optimo_link3_passive, mass 4.310; collision mesh filename=package://meshes/col3.stl; visual mesh filename=package://meshes/link3.stl
- added link optimo_link4, mass 0.0
- added link optimo_link4_passive, mass 1.09; collision mesh filename=package://meshes/col4.stl; visual mesh filename=package://meshes/link4.stl
- added link optimo_link5, mass 0.0
- added link optimo_link5_passive, mass 2.23; collision mesh filename=package://meshes/col5.stl; visual mesh filename=package://meshes/link5.stl
- added link optimo_link6, mass 0.0
- added link optimo_link6_passive, mass 1.138; collision mesh filename=package://meshes/col6.stl; visual mesh filename=package://meshes/link6.stl
- added link optimo_link7, mass 0.0
- added link optimo_link7_passive, mass 1.246; collision mesh filename=package://meshes/col7.stl; visual mesh filename=package://meshes/link7.stl
- added link optimo_pedestal, mass 1.0; collision box size=0.3 0.3 1.0; visual box size=0.3 0.3 1.0
Joints:
- removed joint ee_joint
- removed joint joint1
- removed joint joint1_passive
- removed joint joint2
- removed joint joint2_passive
- removed joint joint3
- removed joint joint3_passive
- removed joint joint4
- removed joint joint4_passive
- removed joint joint5
- removed joint joint5_passive
- removed joint joint6
- removed joint joint6_passive
- removed joint joint7
- removed joint joint7_passive
- removed joint stand_to_link0
- added joint optimo_base_joint: type fixed, parent optimo_base_link, child optimo_link0, origin xyz=0.0 0.0 0.27 rpy=0 0 0
- added joint optimo_ee_joint: type fixed, parent optimo_link7_passive, child optimo_ee_link, origin xyz=0 0 0 rpy=0 0 0
- added joint optimo_joint1: type revolute, parent optimo_link0, child optimo_link1, origin xyz=0 0 0 rpy=0 0 0, axis 0 0 1, limit lower=-2.86233997164 upper=2.91469984917 effort=79 velocity=10
- added joint optimo_joint1_passive: type fixed, parent optimo_link1, child optimo_link1_passive, origin xyz=0 0 0 rpy=1.5707963267948966 0 0
- added joint optimo_joint2: type revolute, parent optimo_link1_passive, child optimo_link2, origin xyz=0 0 0 rpy=0 0 0, axis 0 0 1, limit lower=1.0471975506 upper=4.3633231275 effort=95 velocity=10
- added joint optimo_joint2_passive: type fixed, parent optimo_link2, child optimo_link2_passive, origin xyz=0 0 0 rpy=1.5707963267948966 0 0
- added joint optimo_joint3: type revolute, parent optimo_link2_passive, child optimo_link3, origin xyz=0 0 0.4 rpy=0 0 0, axis 0 0 1, limit lower=-2.91469984917 upper=2.84488667913 effort=32 velocity=10
- added joint optimo_joint3_passive: type fixed, parent optimo_link3, child optimo_link3_passive, origin xyz=0 0 0 rpy=-1.5707963267948966 0 0
- added joint optimo_joint4: type revolute, parent optimo_link3_passive, child optimo_link4, origin xyz=0 0 0 rpy=0 0 0, axis 0 0 1, limit lower=-2.53072741395 upper=2.53072741395 effort=40 velocity=10
- added joint optimo_joint4_passive: type fixed, parent optimo_link4, child optimo_link4_passive, origin xyz=0 0 0 rpy=1.5707963267948966 0 0
- added joint optimo_joint5: type revolute, parent optimo_link4_passive, child optimo_link5, origin xyz=0 0 0.4 rpy=0 0 0, axis 0 0 1, limit lower=-2.9670597267 upper=2.9670597267 effort=15 velocity=10
- added joint optimo_joint5_passive: type fixed, parent optimo_link5, child optimo_link5_passive, origin xyz=0 0 0 rpy=-1.5707963267948966 0 0
- added joint optimo_joint6: type revolute, parent optimo_link5_passive, child optimo_link6, origin xyz=0 0 0 rpy=0 0 0, axis 0 0 1, limit lower=-2.0943951012 upper=2.0943951012 effort=15 velocity=10
- added joint optimo_joint6_passive: type fixed, parent optimo_link6, child optimo_link6_passive, origin xyz=0 0 0 rpy=1.5707963267948966 0 0
- added joint optimo_joint7: type revolute, parent optimo_link6_passive, child optimo_link7, origin xyz=0 0 0 rpy=0 0 0, axis 0 0 1, limit lower=-2.65290046152 upper=3.28121899188 effort=15 velocity=10
- added joint optimo_joint7_passive: type fixed, parent optimo_link7, child optimo_link7_passive, origin xyz=0 0 0 rpy=0 0 0
- added joint optimo_pedestal_joint: type fixed, parent optimo_pedestal, child optimo_base_link, origin xyz=0 0 0.50 rpy=0 0 0

Commit message: plato hand added

File: robot_model/optimo/optimo.urdf (robot description, URDF)
Before this commit: robot optimo, 18 links, 17 joints
Links:
- added link plato_base_link, mass 0.1615803584199397569; collision mesh filename=package://meshes/plato_base_link_collision.stl; visual mesh filename=package://meshes/plato_base_link_visual.stl
- added link plato_bracket_1, mass 0.12656081824380857603; collision mesh filename=package://meshes/plato_bracket_collision.stl; visual mesh filename=package://meshes/plato_bracket_visual.stl
- added link plato_bracket_2, mass 0.12656081824380857603; collision mesh filename=package://meshes/plato_bracket_2_collision.stl; visual mesh filename=package://meshes/plato_bracket_2_visual.stl
- added link plato_bracket_3, mass 0.12656081824380857603; collision mesh filename=package://meshes/plato_bracket_3_collision.stl; visual mesh filename=package://meshes/plato_bracket_3_visual.stl
- added link plato_distal_1, mass 0.0084384550266508422112; collision mesh filename=package://meshes/plato_distal_collision.stl; visual mesh filename=package://meshes/plato_distal_visual.stl
- added link plato_distal_2, mass 0.0084384550266508422112; collision mesh filename=package://meshes/plato_distal_2_collision.stl; visual mesh filename=package://meshes/plato_distal_2_visual.stl
- added link plato_distal_3, mass 0.0084384550266508422112; collision mesh filename=package://meshes/plato_distal_3_collision.stl; visual mesh filename=package://meshes/plato_distal_3_visual.stl
- added link plato_end_effector_1, mass 0.0
- added link plato_end_effector_2, mass 0.0
- added link plato_end_effector_3, mass 0.0
- added link plato_proximal_1, mass 0.069077199724865326336; collision mesh filename=package://meshes/plato_proximal_collision.stl; visual mesh filename=package://meshes/plato_proximal_visual.stl
- added link plato_proximal_2, mass 0.069077199724865326336; collision mesh filename=package://meshes/plato_proximal_2_collision.stl; visual mesh filename=package://meshes/plato_proximal_2_visual.stl
- added link plato_proximal_3, mass 0.069077199724865326336; collision mesh filename=package://meshes/plato_proximal_3_collision.stl; visual mesh filename=package://meshes/plato_proximal_3_visual.stl
Joints:
- added joint plato_connector_joint: type fixed, parent optimo_ee_link, child plato_base_link, origin xyz=0 0 0 rpy=0 0 0
- added joint plato_ee_joint1: type fixed, parent plato_distal_1, child plato_end_effector_1, origin xyz=0.05060 0.0 0.0 rpy=-1.5707 0.0 0.0
- added joint plato_ee_joint2: type fixed, parent plato_distal_2, child plato_end_effector_2, origin xyz=0.05060 0.0 0.0 rpy=-1.5707 0.0 0.0
- added joint plato_ee_joint3: type fixed, parent plato_distal_3, child plato_end_effector_3, origin xyz=0.05060 0.0 0.0 rpy=-1.5707 0.0 0.0
- added joint plato_joint1: type revolute, parent plato_base_link, child plato_bracket_1, origin xyz=0.086299999999999960076 0.029999999999999440309 -0.031000000000000024064 rpy=1.5707963267948978903 0.00091996263300075529958 1.5707963267948956698, axis 0 0 1, limit lower=-0.1745329251994329478 upper=0.785398163397448279 effort=0.06 velocity=0.0872665
- added joint plato_joint2: type revolute, parent plato_bracket_1, child plato_proximal_1, origin xyz=-0.0050000000000000183187 -0.028149999999999991002 -0.0098999999999999921396 rpy=1.8618779238654332436e-18 -1.570796326794896336 0, axis 0 0 1, limit lower=-1.570796326794896558 upper=0.34906585039886589561 effort=0.06 velocity=0.0872665
- added joint plato_joint3: type revolute, parent plato_proximal_1, child plato_distal_1, origin xyz=0.048000000000000000999 2.7755575615628913511e-17 -0.0027000000000001571354 rpy=7.3221470748390791342e-17 1.1335692351879312086e-16 -5.540689055843304715e-17, axis 0 0 1, limit lower=0.0 upper=1.570796326794896558 effort=0.06 velocity=0.0872665
- added joint plato_joint4: type revolute, parent plato_base_link, child plato_bracket_2, origin xyz=0.08399999999999986644 0.029999999999999422962 -0.010000000000000045311 rpy=-3.1415926535897922278 -1.5612511283791256454e-16 1.5655578416789037721, axis 0 0 1, limit lower=-0.087266462599716473902 upper=0.087266462599716473902 effort=0.06 velocity=0.0872665
- added joint plato_joint5: type revolute, parent plato_bracket_2, child plato_proximal_2, origin xyz=-0.004999999999999539535 0.028149999999999578137 -0.0098999999999999799966 rpy=-1.5707963267948972241 4.9960036108132044319e-16 1.5707963267948961139, axis 0 0 1, limit lower=-0.87266462599716476678 upper=0.87266462599716476678 effort=0.06 velocity=0.0872665
- added joint plato_joint6: type revolute, parent plato_proximal_2, child plato_distal_2, origin xyz=0.04800000000000018141 4.4980837630992365206e-17 -0.0029000000000003675615 rpy=1.280885172630899511e-14 -7.2307898014349294445e-15 -1.0713652187632538156e-14, axis 0 0 1, limit lower=-1.570796326794896558 upper=0.0 effort=0.06 velocity=0.0872665
- added joint plato_joint7: type revolute, parent plato_base_link, child plato_bracket_3, origin xyz=0.08399999999999986644 -0.030000000000000463796 -0.010000000000000050515 rpy=-3.1415926535897917837 -9.7144514654701000072e-17 1.5655578416789044383, axis 0 0 1, limit lower=-0.087266462599716473902 upper=0.087266462599716473902 effort=0.06 velocity=0.0872665
- added joint plato_joint8: type revolute, parent plato_bracket_3, child plato_proximal_3, origin xyz=-0.0050000000000000044409 0.028149999999999952838 -0.0099000000000000112216 rpy=-1.570796326794896558 4.9960036108133148724e-16 1.5707963267949323072, axis 0 0 1, limit lower=-0.87266462599716476678 upper=0.87266462599716476678 effort=0.06 velocity=0.0872665
- added joint plato_joint9: type revolute, parent plato_proximal_3, child plato_distal_3, origin xyz=0.047999999999999709566 -1.6328084717631696776e-16 -0.0029000000000011100232 rpy=8.673424925565731141e-16 3.5169650820948147417e-14 -1.6319559976759880709e-29, axis 0 0 1, limit lower=-1.570796326794896558 upper=0.0 effort=0.06 velocity=0.0872665
- joint optimo_ee_joint: origin xyz=0 0 0 rpy=0 0 0 -> xyz=0 0 0.15 rpy=0 -1.5707 3.14

Commit message: remove hand-related variables and add misc variables needed for controller

File: robot_model/optimo/optimo.urdf (robot description, URDF)
Before this commit: robot optimo, 31 links, 30 joints
Joints:
- joint plato_joint1: type revolute -> fixed
- joint plato_joint2: type revolute -> fixed
- joint plato_joint3: type revolute -> fixed
- joint plato_joint4: type revolute -> fixed
- joint plato_joint5: type revolute -> fixed
- joint plato_joint6: type revolute -> fixed
- joint plato_joint7: type revolute -> fixed
- joint plato_joint8: type revolute -> fixed
- joint plato_joint9: type revolute -> fixed
